Commit message: Control, orden, limpieza y script para Jetson

File: src/mi_rover_description/urdf/brazo.urdf (robot description, URDF)
Before this commit: robot brazo_2, 6 links, 5 joints
Joints:
- joint Joint_1: limit lower=-3.1416 upper=3.1416 effort=17.45 velocity=37.7 -> effort=33.6 velocity=1.23; type revolute -> continuous
- joint Joint_2: limit lower=-1.5708 upper=1.5708 effort=45.0 velocity=2.69 -> effort=37.0 velocity=3.67; type revolute -> continuous
- joint Joint_3: limit lower=-3.1416 upper=3.1416 effort=61.0 velocity=5.62 -> lower=-3.1416 upper=3.1416 effort=37.0 velocity=3.67
- joint Joint_4: limit lower=-3.1416 upper=3.1416 effort=15.0 velocity=30.0 -> lower=-3.1416 upper=3.1416 effort=33.6 velocity=1.23

File: src/mi_rover_description/urdf/rover_completo.urdf.xacro (robot description, xacro)
@@ -43,6 +43,9 @@
   <!-- PUBLICADOR DE ESTADOS -->
   <gazebo>
+    <!-- 200 Hz = frecuencia del lazo ADRC. A 50 Hz la medición llega con
+         hasta 20 ms de retraso y el lazo (observador a 50 rad/s) se vuelve
+         inestable, sobre todo con el brazo estirado. -->
     <plugin filename="gz-sim-joint-state-publisher-system" name="gz::sim::systems::JointStatePublisher">
-      <update_rate>50</update_rate>
+      <update_rate>200</update_rate>
       <joint_name>Joint_1</joint_name>
       <joint_name>Joint_2</joint_name>
