Commit message: Fase a: configuración por articulación, perfiles y modelo con articulaciones ausentes
- Perfil del brazo (config/brazos) + plataforma sim/real por capas; n sale del perfil.
- Estados activa/bloqueada/ausente; modelo reducido con pinocchio.buildReducedModel.
- Encoders incrementales (por defecto en el robot) o absolutos por articulación.
- Gazebo: puente ros_gz_bridge en el launch, montadas:=N y escala_masa.

Co-Authored-By: Claude Opus 5.5 <noreply@anthropic.com>
Claude-Session: https://claude.ai/code/session_01HxDsGBVJh5Yv1SVrc6BFFJ

File: src/mi_rover_description/urdf/rover_completo.urdf.xacro (robot description, xacro)
@@ -1,4 +1,12 @@
 <?xml version="1.0"?>
 <robot name="mi_rover_tesis" xmlns:xacro="http://ros.org/wiki/xacro">
+  <!-- ARGUMENTOS DEL BRAZO (ver launch/gazebo.launch.py)
+       montadas:    número de articulaciones montadas (1..5); las demás y
+                    sus eslabones no existen en la simulación.
+       escala_masa: factor de masa e inercia de los eslabones del brazo
+                    (pruebas de robustez del control). -->
+  <xacro:arg name="montadas" default="5"/>
+  <xacro:arg name="escala_masa" default="1.0"/>
+  <xacro:property name="montadas" value="$(arg montadas)"/>
   <!-- INCLUDES PRINCIPALES -->
   <xacro:include filename="$(find mi_rover_description)/urdf/chasis.urdf" />
@@ -10,5 +18,6 @@
   <xacro:llanta prefijo="trasera_der" x="-0.3437" y="-0.315" z="0.15" roll="0" pitch="0" yaw="0" />
   <!-- INCLUIR EL BRAZO -->
-  <xacro:include filename="$(find mi_rover_description)/urdf/brazo.urdf" />
+  <!-- brazo_gz.urdf.xacro se genera de brazo.urdf con scripts/generar_brazo_gz.py -->
+  <xacro:include filename="$(find mi_rover_description)/urdf/brazo_gz.urdf.xacro" />
   <!-- UNION FIJA CHASIS-BRAZO -->
   <joint name="chasis_a_brazo_joint" type="fixed">
@@ -49,8 +58,8 @@
       <update_rate>200</update_rate>
       <joint_name>Joint_1</joint_name>
-      <joint_name>Joint_2</joint_name>
-      <joint_name>Joint_3</joint_name>
-      <joint_name>Joint_4</joint_name>
-      <joint_name>Joint_5</joint_name>
+      <xacro:if value="${montadas >= 2}"><joint_name>Joint_2</joint_name></xacro:if>
+      <xacro:if value="${montadas >= 3}"><joint_name>Joint_3</joint_name></xacro:if>
+      <xacro:if value="${montadas >= 4}"><joint_name>Joint_4</joint_name></xacro:if>
+      <xacro:if value="${montadas >= 5}"><joint_name>Joint_5</joint_name></xacro:if>
     </plugin>
   </gazebo>
@@ -59,26 +68,34 @@
     <plugin filename="mi_rover_initial_pose" name="mi_rover::InitialJointPositions">
       <joint name="Joint_1">3.1415</joint>
-      <joint name="Joint_2">-1.5707</joint>
-      <joint name="Joint_3">0.0</joint>
-      <joint name="Joint_4">0.0</joint>
+      <xacro:if value="${montadas >= 2}"><joint name="Joint_2">-1.5707</joint></xacro:if>
+      <xacro:if value="${montadas >= 3}"><joint name="Joint_3">0.0</joint></xacro:if>
+      <xacro:if value="${montadas >= 4}"><joint name="Joint_4">0.0</joint></xacro:if>
     </plugin>
   </gazebo>
-<!-- CONTROL DE TORQUE PURO PARA J1, J2, J3 -->
+<!-- CONTROL DE TORQUE PURO (una por articulación montada) -->
   <gazebo>
     <plugin filename="gz-sim-apply-joint-force-system" name="gz::sim::systems::ApplyJointForce">
       <joint_name>Joint_1</joint_name>
     </plugin>
+    <xacro:if value="${montadas >= 2}">
     <plugin filename="gz-sim-apply-joint-force-system" name="gz::sim::systems::ApplyJointForce">
       <joint_name>Joint_2</joint_name>
     </plugin>
+    </xacro:if>
+    <xacro:if value="${montadas >= 3}">
     <plugin filename="gz-sim-apply-joint-force-system" name="gz::sim::systems::ApplyJointForce">
       <joint_name>Joint_3</joint_name>
     </plugin>
+    </xacro:if>
+    <xacro:if value="${montadas >= 4}">
     <plugin filename="gz-sim-apply-joint-force-system" name="gz::sim::systems::ApplyJointForce">
       <joint_name>Joint_4</joint_name>
     </plugin>
+    </xacro:if>
+    <xacro:if value="${montadas >= 5}">
     <plugin filename="gz-sim-apply-joint-force-system" name="gz::sim::systems::ApplyJointForce">
       <joint_name>Joint_5</joint_name>
     </plugin>
+    </xacro:if>
   </gazebo>
   <!-- FRICCIÓN DE LAS LLANTAS (Para que el rover se ancle al piso) -->
